Commit message: add fast altas models

File: examples/examples_files/humanoid.urdf (robot description, URDF)
Before this commit: robot atlas, 13 links, 12 joints
Joints:
- joint abdomen_yz: axis 0.00000 0.00000 1.00000 -> 1.00000 0.00000 0.00000; type continuous -> orbital
- joint left_ankle_y: axis 0.00000 1.00000 0.00000 -> -0.44721 0.00000 0.89442
- joint left_shoulder1: axis 2.00000 -1.00000 1.00000 -> 0.57735 0.57735 -0.57735; type ball -> orbital
- joint right_ankle_y: axis 0.00000 1.00000 0.00000 -> -0.44721 0.00000 0.89442
- joint right_shoulder1: axis 2.00000 1.00000 1.00000 -> -0.57735 0.57735 0.57735; type ball -> orbital
