Commit message: trying to fix momentum

File: examples/examples_files/walker2d.urdf (robot description, URDF)
Before this commit: robot walker2d, 17 links, 16 joints
Links:
- removed link foot
- removed link foot_left
- removed link leg
- removed link leg_left
- removed link link0_1
- removed link link0_10
- removed link link0_12
- removed link link0_14
- removed link link0_16
- removed link link0_2
- removed link link0_3
- removed link link0_4
- removed link link0_6
- removed link link0_8
- removed link thigh_left
- link thigh: geometry collision capsule length=0.45000 radius=0.05000; visual cylinder length=0.45000 radius=0.05000
- link torso: geometry collision capsule length=0.40000 radius=0.05000; visual cylinder length=0.40000 radius=0.05000
Joints:
- removed joint foot_joint
- removed joint foot_left_joint
- removed joint ignorex
- removed joint ignorey
- removed joint ignorez
- removed joint jointfix_0_10
- removed joint jointfix_1_8
- removed joint jointfix_2_6
- removed joint jointfix_3_16
- removed joint jointfix_4_14
- removed joint jointfix_5_12
- removed joint jointfix_6_4
- removed joint leg_joint
- removed joint leg_left_joint
- removed joint thigh_left_joint
- joint thigh_joint: child link0_6 -> thigh; origin xyz=0.00000 0.00000 1.05000 rpy=0.00000 -0.00000 0.00000 -> xyz=0.00000 0.00000 0.82500 rpy=0.00000 -0.00000 0.00000
