Commit message: adding halfcheetah all tests are passing

File: examples/examples_files/halfcheetah_pybullet.urdf (robot description, URDF)
Before this commit: robot cheetah, 8 links, 7 joints
Links:
- link bshin: geometry collision capsule length=0.30000 radius=0.04600; visual cylinder length=0.30000 radius=0.04600
Joints:
- joint bfoot: origin xyz=-0.00000 0.00000 -0.29000 rpy=0.00000 -0.00000 0.00000 -> xyz=-0.28000 0.00000 -0.14000 rpy=0.00000 -0.00000 0.00000
- joint bshin: origin xyz=0.0000 0.00000 -0.29000 rpy=0.00000 -0.00000 0.00000 -> xyz=0.16000 0.00000 -0.25000 rpy=0.00000 -0.00000 0.00000
- joint bthigh: origin xyz=-0.50000 0.00000 0.00000 rpy=0.00000 -0.65800 0.00000 -> xyz=-0.50000 0.00000 0.00000 rpy=0.00000 -0.00000 0.00000
- joint ffoot: origin xyz=0.00000 0.00000 -0.21200 rpy=0.00000 -0.00000 0.00000 -> xyz=0.13000 0.00000 -0.18000 rpy=0.00000 -0.00000 0.00000
- joint fshin: origin xyz=-0.00000 0.00000 -0.26600 rpy=0.00000 -1.11159 0.00000 -> xyz=-0.14000 0.00000 -0.24000 rpy=0.00000 -0.00000 0.00000
- joint fthigh: origin xyz=0.50000 0.00000 0.00000 rpy=0.00000 0.52000 0.00000 -> xyz=0.50000 0.00000 0.00000 rpy=0.00000 -0.00000 0.00000
