Commit message: add max2min

File: examples/examples_files/halfcheetah.urdf (robot description, URDF)
Before this commit: robot cheetah, 8 links, 7 joints
Links:
- link bfoot: mass 10.00000 -> 1.069
- link bshin: mass 2.40200 -> 1.5809
- link bthigh: mass 2.33553 -> 1.5352
- link ffoot: mass 10.00000 -> 0.84986
- link fshin: mass 1.81701 -> 1.17885
- link fthigh: mass 2.17598 -> 1.42558
- link torso: mass 9.45733 -> 6.36031
Joints:
- joint bfoot: origin xyz=-0.00000 0.00000 -0.29000 rpy=0.00000 -0.00000 0.00000 -> xyz=-0.00000 0.00000 -0.29000 rpy=0.00000 -1.5 0.00000
- joint bshin: origin xyz=0.0000 0.00000 -0.29000 rpy=0.00000 -0.00000 0.00000 -> xyz=0.0000 0.00000 -0.29000 rpy=0.00000 1.7 0.00000
- joint ffoot: origin xyz=0.00000 0.00000 -0.21200 rpy=0.00000 -0.00000 0.00000 -> xyz=0.00000 0.00000 -0.21200 rpy=0.00000 -0.10000 0.00000
