Commit message: capsule shape

File: env/halfcheetah/deps/halfcheetah.urdf (robot description, URDF)
Before this commit: robot cheetah, 8 links, 7 joints
Links:
- link bfoot: geometry collision capsule length=0.18800 radius=0.04600; visual capsule length=0.18800 radius=0.04600
- link bshin: geometry collision capsule length=0.30000 radius=0.04600; visual capsule length=0.29000 radius=0.04600
- link bthigh: geometry collision capsule length=0.29000 radius=0.04600; visual capsule length=0.29000 radius=0.04600
- link ffoot: geometry collision capsule length=0.14000 radius=0.04600; visual capsule length=0.14000 radius=0.04600
- link fshin: geometry collision capsule length=0.21200 radius=0.04600; visual capsule length=0.21200 radius=0.04600
- link fthigh: geometry collision capsule length=0.26600 radius=0.04600; visual capsule length=0.26600 radius=0.04600
- link torso: geometry collision capsule length=0.30000 radius=0.04600; collision capsule length=1.00000 radius=0.04600
