Commit message: ant env

File: env/ant/deps/ant.urdf (robot description, URDF)
Before this commit: robot ant, 21 links, 20 joints
Links:
- removed link link0_10
- removed link link0_13
- removed link link0_15
- removed link link0_18
- removed link link0_20
- removed link link0_3
- removed link link0_5
- removed link link0_8
- link aux_1: mass 7.83155 -> 0.03647692799740343; geometry collision capsule length=0.28284 radius=0.08000; visual capsule length=0.28284 radius=0.08000
- link aux_2: mass 7.83155 -> 0.03647692799740343; geometry collision capsule length=0.28284 radius=0.08000; visual capsule length=0.28284 radius=0.08000
- link aux_3: mass 7.83155 -> 0.03647692799740343; geometry collision capsule length=0.28284 radius=0.08000; visual capsule length=0.28284 radius=0.08000
- link aux_4: mass 7.83155 -> 0.03647692799740343; geometry collision capsule length=0.28284 radius=0.08000; visual capsule length=0.28284 radius=0.08000
- link front_left_foot: mass 13.51844 -> 0.06491137880161697; geometry collision capsule length=0.56569 radius=0.08000; visual capsule length=0.56569 radius=0.08000
- link front_left_leg: mass 7.83155 -> 0.03647692799740343; geometry collision capsule length=0.28284 radius=0.08000; visual capsule length=0.28284 radius=0.08000
- link front_right_foot: mass 13.51844 -> 0.06491137880161697; geometry collision capsule length=0.56569 radius=0.08000; visual capsule length=0.56569 radius=0.08000
- link front_right_leg: mass 7.83155 -> 0.03647692799740343; geometry collision capsule length=0.28284 radius=0.08000; visual capsule length=0.28284 radius=0.08000
- link left_back_foot: mass 13.51844 -> 0.06491137880161697; geometry collision capsule length=0.56569 radius=0.08000; visual capsule length=0.56569 radius=0.08000
- link left_back_leg: mass 7.83155 -> 0.03647692799740343; geometry collision capsule length=0.28284 radius=0.08000; visual capsule length=0.28284 radius=0.08000
- link right_back_foot: mass 13.51844 -> 0.06491137880161697; geometry collision capsule length=0.56569 radius=0.08000; visual capsule length=0.56569 radius=0.08000
- link right_back_leg: mass 7.83155 -> 0.03647692799740343; geometry collision capsule length=0.28284 radius=0.08000; visual capsule length=0.28284 radius=0.08000
- link torso: mass 65.44985 -> 0.32724923474893675; geometry collision sphere radius=0.25000; visual sphere radius=0.25000
Joints:
- removed joint jointfix_10_18
- removed joint jointfix_11_0
- removed joint jointfix_1_3
- removed joint jointfix_2_0
- removed joint jointfix_4_8
- removed joint jointfix_5_0
- removed joint jointfix_7_13
- removed joint jointfix_8_0
- joint ankle_1: child link0_5 -> aux_1; parent aux_1 -> front_left_leg
- joint ankle_2: child link0_10 -> aux_2; parent aux_2 -> front_right_leg
- joint ankle_3: child link0_15 -> aux_3; parent aux_3 -> left_back_leg
- joint ankle_4: child link0_20 -> aux_4; parent aux_4 -> right_back_leg
- joint hip_1: child link0_3 -> front_left_leg; parent front_left_leg -> torso
- joint hip_2: child link0_8 -> front_right_leg; parent front_right_leg -> torso
- joint hip_3: child link0_13 -> left_back_leg; parent left_back_leg -> torso
- joint hip_4: child link0_18 -> right_back_leg; parent right_back_leg -> torso
- joint jointfix_0_5: parent link0_5 -> aux_1
- joint jointfix_3_10: parent link0_10 -> aux_2
- joint jointfix_6_15: parent link0_15 -> aux_3
- joint jointfix_9_20: parent link0_20 -> aux_4
