Commit message: multiple shapes per body

File: env/humanoid/deps/humanoid.urdf (robot description, URDF)
Before this commit: robot atlas, 13 links, 12 joints
Links:
- link left_foot: geometry collision capsule length=0.21095 radius=0.02700; collision capsule length=0.21095 radius=0.02700
- link left_lower_arm: geometry collision capsule length=0.27713 radius=0.03100; collision sphere radius=0.04000
- link left_shin: geometry collision capsule length=0.30000 radius=0.04900; visual capsule length=0.30000 radius=0.04900
- link left_thigh: geometry collision capsule length=0.34015 radius=0.06000; visual capsule length=0.34015 radius=0.06000
- link left_upper_arm: geometry collision capsule length=0.27713 radius=0.04000; visual capsule length=0.27713 radius=0.04000
- link lwaist: geometry collision capsule length=0.12000 radius=0.06000; visual capsule length=0.12000 radius=0.06000
- link pelvis: geometry collision capsule length=0.14000 radius=0.09000; visual capsule length=0.14000 radius=0.09000
- link right_foot: geometry collision capsule length=0.21095 radius=0.02700; collision capsule length=0.21095 radius=0.02700
- link right_lower_arm: geometry collision capsule length=0.27713 radius=0.03100; collision sphere radius=0.04000
- link right_shin: geometry collision capsule length=0.30000 radius=0.04900; visual capsule length=0.30000 radius=0.04900
- link right_thigh: geometry collision capsule length=0.34015 radius=0.06000; visual capsule length=0.34015 radius=0.06000
- link right_upper_arm: geometry collision capsule length=0.27713 radius=0.04000; visual capsule length=0.27713 radius=0.04000
- link torso: geometry collision capsule length=0.12000 radius=0.06000; collision capsule length=0.14000 radius=0.07000

Commit message: adding regularization

File: env/humanoid/deps/humanoid.urdf (robot description, URDF)
Before this commit: robot atlas, 13 links, 12 joints
Links:
- link left_foot: geometry collision capsule length=0.21095 radius=0.02700; collision capsule length=0.21095 radius=0.02700
