Commit message: finished mujoco hopper env

File: env/hopper/deps/hopper.urdf (robot description, URDF)
Before this commit: robot hopper, 5 links, 4 joints
Links:
- removed link bfoot
- removed link bshin
- removed link bthigh
- added link foot, mass 5.08938; collision capsule length=0.39 radius=0.06; visual capsule length=0.39 radius=0.06
- added link leg, mass 2.71433; collision capsule length=0.5 radius=0.04; visual capsule length=0.5 radius=0.04
- added link thigh, mass 3.92699; collision capsule length=0.45 radius=0.05; visual capsule length=0.45 radius=0.05
- link torso: mass 6.36031 -> 3.53429; geometry collision capsule length=0.40000 radius=0.05; visual capsule length=0.40000 radius=0.05
Joints:
- removed joint bfoot
- removed joint bshin
- removed joint bthigh
- added joint foot: type revolute, parent leg, child foot, origin xyz=0.00000 0.00000 -0.50000 rpy=0.00000 0.00000 0.00000, axis 0.00000 1.00000 0.00000
- added joint leg: type revolute, parent thigh, child leg, origin xyz=0.0000 0.00000 -0.45000 rpy=0.00000 0.00000 0.00000, axis 0.00000 1.00000 0.00000
- added joint thigh: type revolute, parent torso, child thigh, origin xyz=0.00000 0.00000 -0.20000 rpy=0.00000 0.00000 0.00000, axis 0.00000 1.00000 0.00000
- joint floating_joint: origin xyz=0.00000 0.00000 0.00000 rpy=0.00000 -0.00000 0.00000 -> xyz=0.00000 0.00000 0.00000 rpy=0.00000 0.00000 0.00000
