Commit message: atlas + ilqr = 3 steps

File: env/atlas/deps/atlas_armless_old.urdf (robot description, URDF)
Before this commit: robot atlas, 8 links, 7 joints
Joints:
- joint back_bkxyz: child pelvis -> utorso; origin xyz=0.0125 0 -0.212 rpy=0 0 0 -> xyz=-0.0125 0 0.212 rpy=0 0 0; parent utorso -> pelvis
