Commit message: mehrotra solver options

File: env/atlas/deps/atlas_armless.urdf (robot description, URDF)
Before this commit: robot atlas, 8 links, 7 joints
Links:
- link l_foot: geometry visual mesh filename=env/atlas/deps/mesh/l_foot.obj; visual sphere radius=0.01
- link l_lleg: geometry visual mesh filename=env/atlas/deps/mesh/l_lleg.obj
- link l_uleg: geometry visual mesh filename=env/atlas/deps/mesh/l_uleg.obj
- link pelvis: geometry visual mesh filename=env/atlas/deps/mesh/pelvis.obj
- link r_foot: geometry visual mesh filename=env/atlas/deps/mesh/r_foot.obj; visual sphere radius=0.01
- link r_lleg: geometry visual mesh filename=env/atlas/deps/mesh/r_lleg.obj
- link r_uleg: geometry visual mesh filename=env/atlas/deps/mesh/r_uleg.obj
- link utorso: geometry visual mesh filename=env/atlas/deps/mesh/utorso.obj

File: env/atlas/deps/atlas_complex.urdf (robot description, URDF)
Before this commit: robot atlas, 70 links, 69 joints
Links:
- link head: geometry collision mesh filename=env/atlas/deps/mesh/head_chull.obj; visual mesh filename=env/atlas/deps/mesh/head_chull.obj
- link hokuyo_link: geometry collision mesh filename=env/atlas/deps/mesh/head_camera_chull.obj; visual mesh filename=env/atlas/deps/mesh/head_camera_chull.obj
- link l_clav: geometry collision mesh filename=env/atlas/deps/mesh/r_clav_chull.obj; visual mesh filename=env/atlas/deps/mesh/r_clav.obj
- link l_foot: geometry collision mesh filename=env/atlas/deps/mesh/l_foot_chull.obj; collision sphere radius=0.0
- link l_larm: geometry collision mesh filename=env/atlas/deps/mesh/r_larm_chull.obj; visual mesh filename=env/atlas/deps/mesh/r_larm.obj
- link l_lfarm: geometry collision mesh filename=env/atlas/deps/mesh/r_hand_chull.obj; visual mesh filename=env/atlas/deps/mesh/r_hand.obj
- link l_lglut: geometry collision mesh filename=env/atlas/deps/mesh/l_lglut_chull.obj; visual mesh filename=env/atlas/deps/mesh/l_lglut.obj
- link l_lleg: geometry collision mesh filename=env/atlas/deps/mesh/l_lleg_chull.obj; visual mesh filename=env/atlas/deps/mesh/l_lleg.obj
- link l_scap: geometry collision mesh filename=env/atlas/deps/mesh/r_scap_chull.obj; visual mesh filename=env/atlas/deps/mesh/r_scap.obj
- link l_talus: geometry visual mesh filename=env/atlas/deps/mesh/l_talus.obj
- link l_uarm: geometry collision mesh filename=env/atlas/deps/mesh/r_uarm_chull.obj; visual mesh filename=env/atlas/deps/mesh/r_uarm.obj
- link l_ufarm: geometry collision mesh filename=env/atlas/deps/mesh/r_farm_chull.obj; visual mesh filename=env/atlas/deps/mesh/r_farm.obj
- link l_uglut: geometry collision mesh filename=env/atlas/deps/mesh/l_uglut_chull.obj; visual mesh filename=env/atlas/deps/mesh/l_uglut.obj
- link l_uleg: geometry collision mesh filename=env/atlas/deps/mesh/l_uleg_chull.obj; visual mesh filename=env/atlas/deps/mesh/l_uleg.obj
- link left_palm: geometry collision mesh filename=env/atlas/deps/mesh/GRIPPER_OPEN_chull.obj scale=1 1 1; visual mesh filename=env/atlas/deps/mesh/GRIPPER_OPEN_chull.obj scale=1 1 1
- link ltorso: geometry visual mesh filename=env/atlas/deps/mesh/ltorso.obj
- link mtorso: geometry visual mesh filename=env/atlas/deps/mesh/mtorso.obj
- link pelvis: geometry collision mesh filename=env/atlas/deps/mesh/pelvis_chull.obj; visual mesh filename=env/atlas/deps/mesh/pelvis.obj
- link r_clav: geometry collision mesh filename=env/atlas/deps/mesh/r_clav_chull.obj; visual mesh filename=env/atlas/deps/mesh/r_clav.obj
- link r_foot: geometry collision mesh filename=env/atlas/deps/mesh/r_foot_chull.obj; collision sphere radius=0.0
- link r_larm: geometry collision mesh filename=env/atlas/deps/mesh/r_larm_chull.obj; visual mesh filename=env/atlas/deps/mesh/r_larm.obj
- link r_lfarm: geometry collision mesh filename=env/atlas/deps/mesh/r_hand_chull.obj; visual mesh filename=env/atlas/deps/mesh/r_hand.obj
- link r_lglut: geometry collision mesh filename=env/atlas/deps/mesh/r_lglut_chull.obj; visual mesh filename=env/atlas/deps/mesh/r_lglut.obj
- link r_lleg: geometry collision mesh filename=env/atlas/deps/mesh/r_lleg_chull.obj; visual mesh filename=env/atlas/deps/mesh/r_lleg.obj
- link r_scap: geometry collision mesh filename=env/atlas/deps/mesh/r_scap_chull.obj; visual mesh filename=env/atlas/deps/mesh/r_scap.obj
- link r_talus: geometry visual mesh filename=env/atlas/deps/mesh/r_talus.obj
- link r_uarm: geometry collision mesh filename=env/atlas/deps/mesh/r_uarm_chull.obj; visual mesh filename=env/atlas/deps/mesh/r_uarm.obj
- link r_ufarm: geometry collision mesh filename=env/atlas/deps/mesh/r_farm_chull.obj; visual mesh filename=env/atlas/deps/mesh/r_farm.obj
- link r_uglut: geometry collision mesh filename=env/atlas/deps/mesh/r_uglut_chull.obj; visual mesh filename=env/atlas/deps/mesh/r_uglut.obj
- link r_uleg: geometry collision mesh filename=env/atlas/deps/mesh/r_uleg_chull.obj; visual mesh filename=env/atlas/deps/mesh/r_uleg.obj
- link right_palm: geometry collision mesh filename=env/atlas/deps/mesh/GRIPPER_OPEN_chull.obj scale=1 1 1; visual mesh filename=env/atlas/deps/mesh/GRIPPER_OPEN_chull.obj scale=1 1 1
- link utorso: geometry collision mesh filename=env/atlas/deps/mesh/utorso_chull.obj; visual mesh filename=env/atlas/deps/mesh/utorso.obj

File: env/atlas/deps/atlas_debug.urdf (robot description, URDF)
Before this commit: robot atlas, 3 links, 2 joints
Links:
- link ltorso: geometry visual mesh filename=env/atlas/deps/mesh/ltorso.obj
- link mtorso: geometry visual mesh filename=env/atlas/deps/mesh/mtorso.obj
- link pelvis: geometry visual mesh filename=env/atlas/deps/mesh/pelvis.obj

File: env/atlas/deps/atlas_fast.urdf (robot description, URDF)
Before this commit: robot atlas, 23 links, 22 joints
Links:
- link head: geometry visual mesh filename=env/atlas/deps/mesh/head_chull.obj
- link l_clav: geometry visual mesh filename=env/atlas/deps/mesh/r_clav.obj
- link l_foot: geometry visual mesh filename=env/atlas/deps/mesh/l_foot.obj; visual sphere radius=0.01
- link l_larm: geometry visual mesh filename=env/atlas/deps/mesh/r_larm.obj
- link l_lfarm: geometry visual mesh filename=env/atlas/deps/mesh/r_hand.obj
- link l_lleg: geometry visual mesh filename=env/atlas/deps/mesh/l_lleg.obj
- link l_scap: geometry visual mesh filename=env/atlas/deps/mesh/r_scap.obj
- link l_uarm: geometry visual mesh filename=env/atlas/deps/mesh/r_uarm.obj
- link l_ufarm: geometry visual mesh filename=env/atlas/deps/mesh/r_farm.obj
- link l_uleg: geometry visual mesh filename=env/atlas/deps/mesh/l_uleg.obj
- link pelvis: geometry visual mesh filename=env/atlas/deps/mesh/pelvis.obj
- link r_clav: geometry visual mesh filename=env/atlas/deps/mesh/r_clav.obj
- link r_foot: geometry visual mesh filename=env/atlas/deps/mesh/r_foot.obj; visual sphere radius=0.01
- link r_larm: geometry visual mesh filename=env/atlas/deps/mesh/r_larm.obj
- link r_lfarm: geometry visual mesh filename=env/atlas/deps/mesh/r_hand.obj
- link r_lleg: geometry visual mesh filename=env/atlas/deps/mesh/r_lleg.obj
- link r_scap: geometry visual mesh filename=env/atlas/deps/mesh/r_scap.obj
- link r_uarm: geometry visual mesh filename=env/atlas/deps/mesh/r_uarm.obj
- link r_ufarm: geometry visual mesh filename=env/atlas/deps/mesh/r_farm.obj
- link r_uleg: geometry visual mesh filename=env/atlas/deps/mesh/r_uleg.obj
- link utorso: geometry visual mesh filename=env/atlas/deps/mesh/utorso.obj

File: env/atlas/deps/atlas_ones.urdf (robot description, URDF)
Before this commit: robot atlas, 31 links, 30 joints
Links:
- link head: geometry visual mesh filename=env/atlas/deps/mesh/head_chull.obj
- link l_clav: geometry visual mesh filename=env/atlas/deps/mesh/r_clav.obj
- link l_foot: geometry visual mesh filename=env/atlas/deps/mesh/l_foot.obj; visual sphere radius=0.01
- link l_larm: geometry visual mesh filename=env/atlas/deps/mesh/r_larm.obj
- link l_lfarm: geometry visual mesh filename=env/atlas/deps/mesh/r_hand.obj
- link l_lglut: geometry visual mesh filename=env/atlas/deps/mesh/l_lglut.obj
- link l_lleg: geometry visual mesh filename=env/atlas/deps/mesh/l_lleg.obj
- link l_scap: geometry visual mesh filename=env/atlas/deps/mesh/r_scap.obj
- link l_talus: geometry visual mesh filename=env/atlas/deps/mesh/l_talus.obj
- link l_uarm: geometry visual mesh filename=env/atlas/deps/mesh/r_uarm.obj
- link l_ufarm: geometry visual mesh filename=env/atlas/deps/mesh/r_farm.obj
- link l_uglut: geometry visual mesh filename=env/atlas/deps/mesh/l_uglut.obj
- link l_uleg: geometry visual mesh filename=env/atlas/deps/mesh/l_uleg.obj
- link ltorso: geometry visual mesh filename=env/atlas/deps/mesh/ltorso.obj
- link mtorso: geometry visual mesh filename=env/atlas/deps/mesh/mtorso.obj
- link pelvis: geometry visual mesh filename=env/atlas/deps/mesh/pelvis.obj
- link r_clav: geometry visual mesh filename=env/atlas/deps/mesh/r_clav.obj
- link r_foot: geometry visual mesh filename=env/atlas/deps/mesh/r_foot.obj; visual sphere radius=0.01
- link r_larm: geometry visual mesh filename=env/atlas/deps/mesh/r_larm.obj
- link r_lfarm: geometry visual mesh filename=env/atlas/deps/mesh/r_hand.obj
- link r_lglut: geometry visual mesh filename=env/atlas/deps/mesh/r_lglut.obj
- link r_lleg: geometry visual mesh filename=env/atlas/deps/mesh/r_lleg.obj
- link r_scap: geometry visual mesh filename=env/atlas/deps/mesh/r_scap.obj
- link r_talus: geometry visual mesh filename=env/atlas/deps/mesh/r_talus.obj
- link r_uarm: geometry visual mesh filename=env/atlas/deps/mesh/r_uarm.obj
- link r_ufarm: geometry visual mesh filename=env/atlas/deps/mesh/r_farm.obj
- link r_uglut: geometry visual mesh filename=env/atlas/deps/mesh/r_uglut.obj
- link r_uleg: geometry visual mesh filename=env/atlas/deps/mesh/r_uleg.obj
- link utorso: geometry visual mesh filename=env/atlas/deps/mesh/utorso.obj

File: env/atlas/deps/atlas_simple.urdf (robot description, URDF)
Before this commit: robot atlas, 31 links, 30 joints
Links:
- link head: geometry visual mesh filename=env/atlas/deps/mesh/head_chull.obj
- link l_clav: geometry visual mesh filename=env/atlas/deps/mesh/r_clav.obj
- link l_foot: geometry visual mesh filename=env/atlas/deps/mesh/l_foot.obj; visual sphere radius=0.01
- link l_larm: geometry visual mesh filename=env/atlas/deps/mesh/r_larm.obj
- link l_lfarm: geometry visual mesh filename=env/atlas/deps/mesh/r_hand.obj
- link l_lglut: geometry visual mesh filename=env/atlas/deps/mesh/l_lglut.obj
- link l_lleg: geometry visual mesh filename=env/atlas/deps/mesh/l_lleg.obj
- link l_scap: geometry visual mesh filename=env/atlas/deps/mesh/r_scap.obj
- link l_talus: geometry visual mesh filename=env/atlas/deps/mesh/l_talus.obj
- link l_uarm: geometry visual mesh filename=env/atlas/deps/mesh/r_uarm.obj
- link l_ufarm: geometry visual mesh filename=env/atlas/deps/mesh/r_farm.obj
- link l_uglut: geometry visual mesh filename=env/atlas/deps/mesh/l_uglut.obj
- link l_uleg: geometry visual mesh filename=env/atlas/deps/mesh/l_uleg.obj
- link ltorso: geometry visual mesh filename=env/atlas/deps/mesh/ltorso.obj
- link mtorso: geometry visual mesh filename=env/atlas/deps/mesh/mtorso.obj
- link pelvis: geometry visual mesh filename=env/atlas/deps/mesh/pelvis.obj
- link r_clav: geometry visual mesh filename=env/atlas/deps/mesh/r_clav.obj
- link r_foot: geometry visual mesh filename=env/atlas/deps/mesh/r_foot.obj; visual sphere radius=0.01
- link r_larm: geometry visual mesh filename=env/atlas/deps/mesh/r_larm.obj
- link r_lfarm: geometry visual mesh filename=env/atlas/deps/mesh/r_hand.obj
- link r_lglut: geometry visual mesh filename=env/atlas/deps/mesh/r_lglut.obj
- link r_lleg: geometry visual mesh filename=env/atlas/deps/mesh/r_lleg.obj
- link r_scap: geometry visual mesh filename=env/atlas/deps/mesh/r_scap.obj
- link r_talus: geometry visual mesh filename=env/atlas/deps/mesh/r_talus.obj
- link r_uarm: geometry visual mesh filename=env/atlas/deps/mesh/r_uarm.obj
- link r_ufarm: geometry visual mesh filename=env/atlas/deps/mesh/r_farm.obj
- link r_uglut: geometry visual mesh filename=env/atlas/deps/mesh/r_uglut.obj
- link r_uleg: geometry visual mesh filename=env/atlas/deps/mesh/r_uleg.obj
- link utorso: geometry visual mesh filename=env/atlas/deps/mesh/utorso.obj

File: env/quadruped/deps/quadruped_ones.urdf (robot description, URDF)
Before this commit: robot a1_description, 14 links, 13 joints
Links:
- link FL_calf: geometry collision box size=0.2 0.016 0.016; visual mesh filename=env/quadruped/deps/mesh/calf.dae scale=1 1 1
- link FL_hip: geometry collision cylinder length=0.04 radius=0.046; visual mesh filename=env/quadruped/deps/mesh/hip.dae scale=1 1 1
- link FL_thigh: geometry collision box size=0.2 0.0245 0.034; visual mesh filename=env/quadruped/deps/mesh/thigh.dae scale=1 1 1
- link FR_calf: geometry collision box size=0.2 0.016 0.016; visual mesh filename=env/quadruped/deps/mesh/calf.dae scale=1 1 1
- link FR_hip: geometry collision cylinder length=0.04 radius=0.046; visual mesh filename=env/quadruped/deps/mesh/hip.dae scale=1 1 1
- link FR_thigh: geometry collision box size=0.2 0.0245 0.034; visual mesh filename=env/quadruped/deps/mesh/thigh_mirror.dae scale=1 1 1
- link RL_calf: geometry collision box size=0.2 0.016 0.016; visual mesh filename=env/quadruped/deps/mesh/calf.dae scale=1 1 1
- link RL_hip: geometry collision cylinder length=0.04 radius=0.046; visual mesh filename=env/quadruped/deps/mesh/hip.dae scale=1 1 1
- link RL_thigh: geometry collision box size=0.2 0.0245 0.034; visual mesh filename=env/quadruped/deps/mesh/thigh.dae scale=1 1 1
- link RR_calf: geometry collision box size=0.2 0.016 0.016; visual mesh filename=env/quadruped/deps/mesh/calf.dae scale=1 1 1
- link RR_hip: geometry collision cylinder length=0.04 radius=0.046; visual mesh filename=env/quadruped/deps/mesh/hip.dae scale=1 1 1
- link RR_thigh: geometry collision box size=0.2 0.0245 0.034; visual mesh filename=env/quadruped/deps/mesh/thigh_mirror.dae scale=1 1 1
- link trunk: geometry collision box size=0.267 0.194 0.114; visual mesh filename=env/quadruped/deps/mesh/trunk.dae scale=1 1 1

File: env/quadruped/deps/quadruped_simon.urdf (robot description, URDF)
Before this commit: robot a1_description, 13 links, 12 joints
Links:
- link FL_calf: geometry collision box size=0.2 0.016 0.016; visual mesh filename=env/quadruped/deps/mesh/calf.dae scale=1 1 1
- link FL_hip: geometry collision cylinder length=0.04 radius=0.046; visual mesh filename=env/quadruped/deps/mesh/hip.dae scale=1 1 1
- link FL_thigh: geometry collision box size=0.2 0.0245 0.034; visual mesh filename=env/quadruped/deps/mesh/thigh.dae scale=1 1 1
- link FR_calf: geometry collision box size=0.2 0.016 0.016; visual mesh filename=env/quadruped/deps/mesh/calf.dae scale=1 1 1
- link FR_hip: geometry collision cylinder length=0.04 radius=0.046; visual mesh filename=env/quadruped/deps/mesh/hip.dae scale=1 1 1
- link FR_thigh: geometry collision box size=0.2 0.0245 0.034; visual mesh filename=env/quadruped/deps/mesh/thigh_mirror.dae scale=1 1 1
- link RL_calf: geometry collision box size=0.2 0.016 0.016; visual mesh filename=env/quadruped/deps/mesh/calf.dae scale=1 1 1
- link RL_hip: geometry collision cylinder length=0.04 radius=0.046; visual mesh filename=env/quadruped/deps/mesh/hip.dae scale=1 1 1
- link RL_thigh: geometry collision box size=0.2 0.0245 0.034; visual mesh filename=env/quadruped/deps/mesh/thigh.dae scale=1 1 1
- link RR_calf: geometry collision box size=0.2 0.016 0.016; visual mesh filename=env/quadruped/deps/mesh/calf.dae scale=1 1 1
- link RR_hip: geometry collision cylinder length=0.04 radius=0.046; visual mesh filename=env/quadruped/deps/mesh/hip.dae scale=1 1 1
- link RR_thigh: geometry collision box size=0.2 0.0245 0.034; visual mesh filename=env/quadruped/deps/mesh/thigh_mirror.dae scale=1 1 1
- link trunk: geometry collision box size=0.267 0.194 0.114; visual mesh filename=env/quadruped/deps/mesh/trunk.dae scale=1 1 1

File: env/quadruped/deps/quadruped_simple.urdf (robot description, URDF)
Before this commit: robot a1_description, 14 links, 13 joints
Links:
- link FL_calf: geometry collision box size=0.2 0.016 0.016; visual mesh filename=env/quadruped/deps/mesh/calf.dae scale=1 1 1
- link FL_hip: geometry collision cylinder length=0.04 radius=0.046; visual mesh filename=env/quadruped/deps/mesh/hip.dae scale=1 1 1
- link FL_thigh: geometry collision box size=0.2 0.0245 0.034; visual mesh filename=env/quadruped/deps/mesh/thigh.dae scale=1 1 1
- link FR_calf: geometry collision box size=0.2 0.016 0.016; visual mesh filename=env/quadruped/deps/mesh/calf.dae scale=1 1 1
- link FR_hip: geometry collision cylinder length=0.04 radius=0.046; visual mesh filename=env/quadruped/deps/mesh/hip.dae scale=1 1 1
- link FR_thigh: geometry collision box size=0.2 0.0245 0.034; visual mesh filename=env/quadruped/deps/mesh/thigh_mirror.dae scale=1 1 1
- link RL_calf: geometry collision box size=0.2 0.016 0.016; visual mesh filename=env/quadruped/deps/mesh/calf.dae scale=1 1 1
- link RL_hip: geometry collision cylinder length=0.04 radius=0.046; visual mesh filename=env/quadruped/deps/mesh/hip.dae scale=1 1 1
- link RL_thigh: geometry collision box size=0.2 0.0245 0.034; visual mesh filename=env/quadruped/deps/mesh/thigh.dae scale=1 1 1
- link RR_calf: geometry collision box size=0.2 0.016 0.016; visual mesh filename=env/quadruped/deps/mesh/calf.dae scale=1 1 1
- link RR_hip: geometry collision cylinder length=0.04 radius=0.046; visual mesh filename=env/quadruped/deps/mesh/hip.dae scale=1 1 1
- link RR_thigh: geometry collision box size=0.2 0.0245 0.034; visual mesh filename=env/quadruped/deps/mesh/thigh_mirror.dae scale=1 1 1
- link trunk: geometry collision box size=0.267 0.194 0.114; visual mesh filename=env/quadruped/deps/mesh/trunk.dae scale=1 1 1

Commit message: atlas + =ilqr = 6 steps

File: env/atlas/deps/atlas_armless.urdf (robot description, URDF)
Before this commit: robot atlas, 8 links, 7 joints
Links:
- added link base, mass 1.00000
Joints:
- added joint auto_generated_floating_joint: type floating, parent base, child utorso, origin xyz=0.00000 0.00000 0.00000 rpy=0.00000 0.00000 0.00000, axis 0.00000 1.00000 0.00000
