Commit message: adding rexhopper and changing urdf parser

File: env/rexhopper/deps/rexhopper.urdf (robot description, URDF)
Before this commit: robot rexhopper, 8 links, 7 joints
Links:
- removed link Link 0
- removed link Link 1
- removed link Link 2
- removed link Link 3
- added link link0, mass 0.256385566503952; collision mesh filename=env/rexhopper/deps/mesh/link0.obj; visual mesh filename=env/rexhopper/deps/mesh/link0.obj
- added link link1, mass 0.0631473819780702; collision mesh filename=env/rexhopper/deps/mesh/link1.obj; visual mesh filename=env/rexhopper/deps/mesh/link1.obj
- added link link2, mass 0.288845046277886; collision mesh filename=env/rexhopper/deps/mesh/link2.obj; visual mesh filename=env/rexhopper/deps/mesh/link2.obj
- added link link3, mass 0.12485760282637; collision mesh filename=env/rexhopper/deps/mesh/link3.obj; visual mesh filename=env/rexhopper/deps/mesh/link3.obj
- link base_link: geometry collision mesh filename=env/rexhopper/deps/mesh/base_link.obj; visual mesh filename=env/rexhopper/deps/mesh/base_link.obj
- link rw0: geometry collision mesh filename=env/rexhopper/deps/mesh/rw0.obj; visual mesh filename=env/rexhopper/deps/mesh/rw0.obj
- link rw1: geometry collision mesh filename=env/rexhopper/deps/mesh/rw1.obj; visual mesh filename=env/rexhopper/deps/mesh/rw1.obj
- link rwz: geometry collision mesh filename=env/rexhopper/deps/mesh/rwz.obj; visual mesh filename=env/rexhopper/deps/mesh/rwz.obj
Joints:
- removed joint Joint 1
- removed joint Joint 2
- removed joint Joint 3
- added joint joint1: type revolute, parent link0, child link1, origin xyz=0.0999999999999999 0 0 rpy=-3.14159265358979 1.0768315178335 -3.14159265358979, axis 0 -1 0, limit lower=-0.7597 upper=1.8295 effort=0 velocity=0
- added joint joint2: type revolute, parent base_link, child link2, origin xyz=0 0 0 rpy=3.14159265358979 0.553232742319403 -3.14159265358979, axis 0 -1 0, limit lower=-3.14 upper=3.14 effort=0 velocity=0
- added joint joint4: type revolute, parent link1, child link3, origin xyz=0.3174120461954416  0.0  -0.08804599865731941 rpy=0.0 -2.0647611361516 0.0, axis 0 -1 0, limit lower=-3.14 upper=3.14 effort=0 velocity=0
- joint Joint 0: child Link 0 -> link0
