Commit message: working on the graph, test passing

File: env/rexhopper/deps/hopper_rev05_alt.urdf (robot description, URDF)
Before this commit: robot rexhopper, 8 links, 7 joints
Links:
- removed link link0
- removed link link1
- removed link link2
- removed link link3
- added link Link 0, mass 0.256385566503952; collision mesh filename=package://hopper_rev05_alt/meshes/Link 0.STL; visual mesh filename=package://hopper_rev05_alt/meshes/Link 0.STL
- added link Link 1, mass 0.0631473819780702; collision mesh filename=package://hopper_rev05_alt/meshes/Link 1.STL; visual mesh filename=package://hopper_rev05_alt/meshes/Link 1.STL
- added link Link 2, mass 0.288845047026487; collision mesh filename=package://hopper_rev05_alt/meshes/Link 2.STL; visual mesh filename=package://hopper_rev05_alt/meshes/Link 2.STL
- added link Link 3, mass 0.124857597760897; collision mesh filename=package://hopper_rev05_alt/meshes/Link 3.STL; visual mesh filename=package://hopper_rev05_alt/meshes/Link 3.STL
- link base_link: mass 5.59607837933863 -> 5.59607837933722; geometry collision mesh filename=package://hopper_rev05_alt/meshes/base_link.STL; visual mesh filename=package://hopper_rev05_alt/meshes/base_link.STL
- link rw0: mass 0.715641175075329 -> 0.715641175075328; geometry collision mesh filename=package://hopper_rev05_alt/meshes/rw0.STL; visual mesh filename=package://hopper_rev05_alt/meshes/rw0.STL
- link rw1: geometry collision mesh filename=package://hopper_rev05_alt/meshes/rw1.STL; visual mesh filename=package://hopper_rev05_alt/meshes/rw1.STL
- link rwz: geometry collision mesh filename=package://hopper_rev05_alt/meshes/rwz.STL; visual mesh filename=package://hopper_rev05_alt/meshes/rwz.STL
Joints:
- removed joint joint1
- removed joint joint2
- removed joint joint3
- added joint Joint 1: type revolute, parent Link 0, child Link 1, origin xyz=0.1 0 0 rpy=-3.1416 1.0768 -3.1416, axis 0 -1 0, limit lower=-0.7597 upper=1.8295 effort=0 velocity=0
- added joint Joint 2: type revolute, parent base_link, child Link 2, origin xyz=0 0 0 rpy=3.1416 0.55323 -3.1416, axis 0 -1 0, limit lower=-3.14 upper=3.14 effort=0 velocity=0
- added joint Joint 4: type revolute, parent Link 1, child Link 3, origin xyz=0.27 0 0 rpy=-3.1416 -1.0768 3.1416, axis 0 -1 0, limit lower=-1.57 upper=1.57 effort=0 velocity=0
- joint Joint 0: child link0 -> Link 0
- joint joint_rw0: axis 1 0 0 -> -1 0 0; origin xyz=0.0620132647100599 -0.147253675939521 0 rpy=3.03065856040946 0 -0.785398163397452 -> xyz=0.062013 -0.14725 0 rpy=3.0307 0 -0.7854
- joint joint_rw1: origin xyz=0.063525686232125 0.148766097461586 0 rpy=-0.0304329711040608 0 0.785398163397453 -> xyz=0.063526 0.14877 0 rpy=-0.030433 0 0.7854
