Commit message: untested new ordering

File: env/rexhopper/deps/rexhopper_no_wheel.urdf (robot description, URDF)
Before this commit: robot rexhopper, 8 links, 7 joints
Links:
- removed link rw0
- removed link rw1
- removed link rwz
Joints:
- removed joint joint_rw0
- removed joint joint_rw1
- removed joint joint_rwz
