Commit message: cleanup

File: env/fourbar/deps/fourbar.urdf (robot description, URDF)
Before this commit: robot Fourbar, 5 links, 4 joints
Joints:
- removed joint joint13
- added joint jointb3: type continuous, parent base_link, child link3, origin xyz=0 0 2.1 rpy=-0.0 0 0, axis 1 0 0
- joint joint12: origin xyz=0 0 -1 rpy=0.2 0 0 -> xyz=0 0 -1 rpy=0.0 0 0
- joint joint34: origin xyz=0 0 -1 rpy=-0.4 0 0 -> xyz=0 0 -1 rpy=-0.0 0 0
- joint jointb1: origin xyz=0 0 0 rpy=0.1 0 0 -> xyz=0 0 2.1 rpy=0.0 0 0

File: env/fourbar/deps/fourbar_open.urdf (robot description, URDF)
Before this commit: robot Fourbar, 5 links, 4 joints
Joints:
- joint jointb1: origin xyz=0 0 0 rpy=0.0 0 0 -> xyz=0 0 2.1 rpy=0.0 0 0
- joint jointb3: origin xyz=0 0 0 rpy=-0.0 0 0 -> xyz=0 0 2.1 rpy=-0.0 0 0
