Commit message: set_floating_base

File: environments/atlas/deps/atlas_armless.urdf (robot description, URDF)
Before this commit: robot atlas, 9 links, 8 joints
Joints:
- removed joint auto_generated_floating_joint
- added joint floating_base: type floating, parent base, child utorso, origin xyz=0.00000 0.00000 0.00000 rpy=0.00000 0.00000 0.00000, axis 0.00000 1.00000 0.00000
