Commit message: removing dvector_rotatedp

File: environments/panda/deps/panda_end_effector.urdf (robot description, URDF)
Before this commit: robot panda, 2 links, 1 joints
Links:
- removed link panda_link2
- added link finger1, mass 3e-1; collision mesh filename=environments/panda/deps/mesh/collision/finger.stl; visual mesh filename=environments/panda/deps/mesh/visual/finger.dae
- added link finger2, mass 3e-1; collision mesh filename=environments/panda/deps/mesh/collision/finger.stl; visual mesh filename=environments/panda/deps/mesh/visual/finger.dae
- added link link0, mass 0.629769273993887; collision mesh filename=environments/panda/deps/mesh/collision/link0.stl; visual mesh filename=environments/panda/deps/mesh/visual/link0.dae
- added link link1, mass 4.970684; collision mesh filename=environments/panda/deps/mesh/collision/link1.stl; visual mesh filename=environments/panda/deps/mesh/visual/link1.dae
- added link link2, mass 0.646926; collision mesh filename=environments/panda/deps/mesh/collision/link2.stl; visual mesh filename=environments/panda/deps/mesh/visual/link2.dae
- added link link3, mass 3.228604; collision mesh filename=environments/panda/deps/mesh/collision/link3.stl; visual mesh filename=environments/panda/deps/mesh/visual/link3.dae
- added link link4, mass 3.587895; collision mesh filename=environments/panda/deps/mesh/collision/link4.stl; visual mesh filename=environments/panda/deps/mesh/visual/link4.dae
- added link link5, mass 1.225946; collision mesh filename=environments/panda/deps/mesh/collision/link5.stl; visual mesh filename=environments/panda/deps/mesh/visual/link5.dae
- added link link6, mass 1.666555; collision mesh filename=environments/panda/deps/mesh/collision/link6.stl; visual mesh filename=environments/panda/deps/mesh/visual/link6.dae
- added link link7, mass 7.35522e-01; collision mesh filename=environments/panda/deps/mesh/collision/link7.stl; visual mesh filename=environments/panda/deps/mesh/visual/link7.dae
- added link link8, mass 7e-1; collision mesh filename=environments/panda/deps/mesh/collision/hand.stl; visual mesh filename=environments/panda/deps/mesh/visual/hand.dae
Joints:
- removed joint panda_joint2
- added joint joint0: type fixed, parent world, child link0, origin xyz=0 0 0 rpy=0 0 0
- added joint joint1: type revolute, parent link0, child link1, origin xyz=0 0 0.333 rpy=0 0 0, axis 0 0 1, limit lower=-2.9671 upper=2.9671 effort=87 velocity=2.5
- added joint joint2: type revolute, parent link1, child link2, origin xyz=0 0 0 rpy=-1.57079632679 0 0, axis 0 0 1, limit lower=-1.8326 upper=1.8326 effort=87 velocity=2.5
- added joint joint3: type revolute, parent link2, child link3, origin xyz=0 -0.316 0 rpy=1.57079632679 0 0, axis 0 0 1, limit lower=-2.9671 upper=2.9671 effort=87 velocity=2.5
- added joint joint4: type revolute, parent link3, child link4, origin xyz=0.0825 0 0 rpy=1.57079632679 0 0, axis 0 0 1, limit lower=-3.1416 upper=-0.4 effort=87 velocity=2.5
- added joint joint5: type revolute, parent link4, child link5, origin xyz=-0.0825 0.384 0 rpy=-1.57079632679 0 0, axis 0 0 1, limit lower=-2.9671 upper=2.9671 effort=12 velocity=3
- added joint joint6: type revolute, parent link5, child link6, origin xyz=0 0 0 rpy=1.57079632679 0 0, axis 0 0 1, limit lower=-0.0873 upper=3.8223 effort=12 velocity=3
- added joint joint7: type revolute, parent link6, child link7, origin xyz=0.088 0 0 rpy=1.57079632679 0 0, axis 0 0 1, limit lower=-2.9671 upper=2.9671 effort=12 velocity=3
- added joint joint8: type fixed, parent link7, child link8, origin xyz=0 0 0.107 rpy=0 0 0, axis 0 0 0
- added joint jointf1: type prismatic, parent link8, child finger1, origin xyz=0 0 0.0584 rpy=0 0 0, axis 0 1 0, limit lower=0.0 upper=0.04 effort=20 velocity=0.2
- added joint jointf2: type prismatic, parent link8, child finger2, origin xyz=0 0 0.0584 rpy=0 0 0, axis 0 -1 0, limit lower=0.0 upper=0.04 effort=20 velocity=0.2, mimic joint=panda_finger_joint1
