Commit message: get DojoEnvironment tests to pass

File: DojoEnvironments/src/atlas/deps/atlas_armless.urdf (robot description, URDF)
Before this commit: robot atlas, 9 links, 8 joints
Links:
- link l_foot: geometry visual mesh filename=mesh/l_foot.obj; visual sphere radius=0.01
- link l_lleg: geometry visual mesh filename=mesh/l_lleg.obj
- link l_uleg: geometry visual mesh filename=mesh/l_uleg.obj
- link pelvis: geometry visual mesh filename=mesh/pelvis.obj
- link r_foot: geometry visual mesh filename=mesh/r_foot.obj; visual sphere radius=0.01
- link r_lleg: geometry visual mesh filename=mesh/r_lleg.obj
- link r_uleg: geometry visual mesh filename=mesh/r_uleg.obj
- link utorso: geometry visual mesh filename=mesh/utorso.obj

File: DojoEnvironments/src/atlas/deps/atlas_armless_old.urdf (robot description, URDF)
Before this commit: robot atlas, 8 links, 7 joints
Links:
- link l_foot: geometry visual mesh filename=mesh/l_foot.obj; visual sphere radius=0.01
- link l_lleg: geometry visual mesh filename=mesh/l_lleg.obj
- link l_uleg: geometry visual mesh filename=mesh/l_uleg.obj
- link pelvis: geometry visual mesh filename=mesh/pelvis.obj
- link r_foot: geometry visual mesh filename=mesh/r_foot.obj; visual sphere radius=0.01
- link r_lleg: geometry visual mesh filename=mesh/r_lleg.obj
- link r_uleg: geometry visual mesh filename=mesh/r_uleg.obj
- link utorso: geometry visual mesh filename=mesh/utorso.obj

File: DojoEnvironments/src/atlas/deps/atlas_complex.urdf (robot description, URDF)
Before this commit: robot atlas, 70 links, 69 joints
Links:
- link head: geometry collision mesh filename=mesh/head_chull.obj; visual mesh filename=mesh/head_chull.obj
- link hokuyo_link: geometry collision mesh filename=mesh/head_camera_chull.obj; visual mesh filename=mesh/head_camera_chull.obj
- link l_clav: geometry collision mesh filename=mesh/r_clav_chull.obj; visual mesh filename=mesh/r_clav.obj
- link l_foot: geometry collision mesh filename=mesh/l_foot_chull.obj; collision sphere radius=0.0
- link l_larm: geometry collision mesh filename=mesh/r_larm_chull.obj; visual mesh filename=mesh/r_larm.obj
- link l_lfarm: geometry collision mesh filename=mesh/r_hand_chull.obj; visual mesh filename=mesh/r_hand.obj
- link l_lglut: geometry collision mesh filename=mesh/l_lglut_chull.obj; visual mesh filename=mesh/l_lglut.obj
- link l_lleg: geometry collision mesh filename=mesh/l_lleg_chull.obj; visual mesh filename=mesh/l_lleg.obj
- link l_scap: geometry collision mesh filename=mesh/r_scap_chull.obj; visual mesh filename=mesh/r_scap.obj
- link l_talus: geometry visual mesh filename=mesh/l_talus.obj
- link l_uarm: geometry collision mesh filename=mesh/r_uarm_chull.obj; visual mesh filename=mesh/r_uarm.obj
- link l_ufarm: geometry collision mesh filename=mesh/r_farm_chull.obj; visual mesh filename=mesh/r_farm.obj
- link l_uglut: geometry collision mesh filename=mesh/l_uglut_chull.obj; visual mesh filename=mesh/l_uglut.obj
- link l_uleg: geometry collision mesh filename=mesh/l_uleg_chull.obj; visual mesh filename=mesh/l_uleg.obj
- link left_palm: geometry collision mesh filename=mesh/GRIPPER_OPEN_chull.obj scale=1 1 1; visual mesh filename=mesh/GRIPPER_OPEN_chull.obj scale=1 1 1
- link ltorso: geometry visual mesh filename=mesh/ltorso.obj
- link mtorso: geometry visual mesh filename=mesh/mtorso.obj
- link pelvis: geometry collision mesh filename=mesh/pelvis_chull.obj; visual mesh filename=mesh/pelvis.obj
- link r_clav: geometry collision mesh filename=mesh/r_clav_chull.obj; visual mesh filename=mesh/r_clav.obj
- link r_foot: geometry collision mesh filename=mesh/r_foot_chull.obj; collision sphere radius=0.0
- link r_larm: geometry collision mesh filename=mesh/r_larm_chull.obj; visual mesh filename=mesh/r_larm.obj
- link r_lfarm: geometry collision mesh filename=mesh/r_hand_chull.obj; visual mesh filename=mesh/r_hand.obj
- link r_lglut: geometry collision mesh filename=mesh/r_lglut_chull.obj; visual mesh filename=mesh/r_lglut.obj
- link r_lleg: geometry collision mesh filename=mesh/r_lleg_chull.obj; visual mesh filename=mesh/r_lleg.obj
- link r_scap: geometry collision mesh filename=mesh/r_scap_chull.obj; visual mesh filename=mesh/r_scap.obj
- link r_talus: geometry visual mesh filename=mesh/r_talus.obj
- link r_uarm: geometry collision mesh filename=mesh/r_uarm_chull.obj; visual mesh filename=mesh/r_uarm.obj
- link r_ufarm: geometry collision mesh filename=mesh/r_farm_chull.obj; visual mesh filename=mesh/r_farm.obj
- link r_uglut: geometry collision mesh filename=mesh/r_uglut_chull.obj; visual mesh filename=mesh/r_uglut.obj
- link r_uleg: geometry collision mesh filename=mesh/r_uleg_chull.obj; visual mesh filename=mesh/r_uleg.obj
- link right_palm: geometry collision mesh filename=mesh/GRIPPER_OPEN_chull.obj scale=1 1 1; visual mesh filename=mesh/GRIPPER_OPEN_chull.obj scale=1 1 1
- link utorso: geometry collision mesh filename=mesh/utorso_chull.obj; visual mesh filename=mesh/utorso.obj

File: DojoEnvironments/src/atlas/deps/atlas_fast.urdf (robot description, URDF)
Before this commit: robot atlas, 23 links, 22 joints
Links:
- link head: geometry visual mesh filename=mesh/head_chull.obj
- link l_clav: geometry visual mesh filename=mesh/r_clav.obj
- link l_foot: geometry visual mesh filename=mesh/l_foot.obj; visual sphere radius=0.01
- link l_larm: geometry visual mesh filename=mesh/r_larm.obj
- link l_lfarm: geometry visual mesh filename=mesh/r_hand.obj
- link l_lleg: geometry visual mesh filename=mesh/l_lleg.obj
- link l_scap: geometry visual mesh filename=mesh/r_scap.obj
- link l_uarm: geometry visual mesh filename=mesh/r_uarm.obj
- link l_ufarm: geometry visual mesh filename=mesh/r_farm.obj
- link l_uleg: geometry visual mesh filename=mesh/l_uleg.obj
- link pelvis: geometry visual mesh filename=mesh/pelvis.obj
- link r_clav: geometry visual mesh filename=mesh/r_clav.obj
- link r_foot: geometry visual mesh filename=mesh/r_foot.obj; visual sphere radius=0.01
- link r_larm: geometry visual mesh filename=mesh/r_larm.obj
- link r_lfarm: geometry visual mesh filename=mesh/r_hand.obj
- link r_lleg: geometry visual mesh filename=mesh/r_lleg.obj
- link r_scap: geometry visual mesh filename=mesh/r_scap.obj
- link r_uarm: geometry visual mesh filename=mesh/r_uarm.obj
- link r_ufarm: geometry visual mesh filename=mesh/r_farm.obj
- link r_uleg: geometry visual mesh filename=mesh/r_uleg.obj
- link utorso: geometry visual mesh filename=mesh/utorso.obj

File: DojoEnvironments/src/atlas/deps/atlas_ones.urdf (robot description, URDF)
Before this commit: robot atlas, 31 links, 30 joints
Links:
- link head: geometry visual mesh filename=mesh/head_chull.obj
- link l_clav: geometry visual mesh filename=mesh/r_clav.obj
- link l_foot: geometry visual mesh filename=mesh/l_foot.obj; visual sphere radius=0.01
- link l_larm: geometry visual mesh filename=mesh/r_larm.obj
- link l_lfarm: geometry visual mesh filename=mesh/r_hand.obj
- link l_lglut: geometry visual mesh filename=mesh/l_lglut.obj
- link l_lleg: geometry visual mesh filename=mesh/l_lleg.obj
- link l_scap: geometry visual mesh filename=mesh/r_scap.obj
- link l_talus: geometry visual mesh filename=mesh/l_talus.obj
- link l_uarm: geometry visual mesh filename=mesh/r_uarm.obj
- link l_ufarm: geometry visual mesh filename=mesh/r_farm.obj
- link l_uglut: geometry visual mesh filename=mesh/l_uglut.obj
- link l_uleg: geometry visual mesh filename=mesh/l_uleg.obj
- link ltorso: geometry visual mesh filename=mesh/ltorso.obj
- link mtorso: geometry visual mesh filename=mesh/mtorso.obj
- link pelvis: geometry visual mesh filename=mesh/pelvis.obj
- link r_clav: geometry visual mesh filename=mesh/r_clav.obj
- link r_foot: geometry visual mesh filename=mesh/r_foot.obj; visual sphere radius=0.01
- link r_larm: geometry visual mesh filename=mesh/r_larm.obj
- link r_lfarm: geometry visual mesh filename=mesh/r_hand.obj
- link r_lglut: geometry visual mesh filename=mesh/r_lglut.obj
- link r_lleg: geometry visual mesh filename=mesh/r_lleg.obj
- link r_scap: geometry visual mesh filename=mesh/r_scap.obj
- link r_talus: geometry visual mesh filename=mesh/r_talus.obj
- link r_uarm: geometry visual mesh filename=mesh/r_uarm.obj
- link r_ufarm: geometry visual mesh filename=mesh/r_farm.obj
- link r_uglut: geometry visual mesh filename=mesh/r_uglut.obj
- link r_uleg: geometry visual mesh filename=mesh/r_uleg.obj
- link utorso: geometry visual mesh filename=mesh/utorso.obj

File: DojoEnvironments/src/atlas/deps/atlas_simple.urdf (robot description, URDF)
Before this commit: robot atlas, 31 links, 30 joints
Links:
- link head: geometry visual mesh filename=mesh/head.obj
- link l_clav: geometry visual mesh filename=mesh/r_clav.obj
- link l_foot: geometry visual mesh filename=mesh/l_foot.obj; visual sphere radius=0.01
- link l_larm: geometry visual mesh filename=mesh/r_larm.obj
- link l_lfarm: geometry visual mesh filename=mesh/r_hand.obj
- link l_lglut: geometry visual mesh filename=mesh/l_lglut.obj
- link l_lleg: geometry visual mesh filename=mesh/l_lleg.obj
- link l_scap: geometry visual mesh filename=mesh/r_scap.obj
- link l_talus: geometry visual mesh filename=mesh/l_talus.obj
- link l_uarm: geometry visual mesh filename=mesh/r_uarm.obj
- link l_ufarm: geometry visual mesh filename=mesh/r_farm.obj
- link l_uglut: geometry visual mesh filename=mesh/l_uglut.obj
- link l_uleg: geometry visual mesh filename=mesh/l_uleg.obj
- link ltorso: geometry visual mesh filename=mesh/ltorso.obj
- link mtorso: geometry visual mesh filename=mesh/mtorso.obj
- link pelvis: geometry visual mesh filename=mesh/pelvis.obj
- link r_clav: geometry visual mesh filename=mesh/r_clav.obj
- link r_foot: geometry visual mesh filename=mesh/r_foot.obj; visual sphere radius=0.01
- link r_larm: geometry visual mesh filename=mesh/r_larm.obj
- link r_lfarm: geometry visual mesh filename=mesh/r_hand.obj
- link r_lglut: geometry visual mesh filename=mesh/r_lglut.obj
- link r_lleg: geometry visual mesh filename=mesh/r_lleg.obj
- link r_scap: geometry visual mesh filename=mesh/r_scap.obj
- link r_talus: geometry visual mesh filename=mesh/r_talus.obj
- link r_uarm: geometry visual mesh filename=mesh/r_uarm.obj
- link r_ufarm: geometry visual mesh filename=mesh/r_farm.obj
- link r_uglut: geometry visual mesh filename=mesh/r_uglut.obj
- link r_uleg: geometry visual mesh filename=mesh/r_uleg.obj
- link utorso: geometry visual mesh filename=mesh/utorso.obj

File: DojoEnvironments/src/atlas/deps/atlas_v2.urdf (robot description, URDF)
Before this commit: robot atlas, 31 links, 30 joints
Links:
- link head: geometry visual mesh filename=mesh/head.obj
- link l_clav: geometry visual mesh filename=mesh/r_clav.obj
- link l_foot: geometry visual mesh filename=mesh/l_foot.obj
- link l_larm: geometry visual mesh filename=mesh/r_larm.obj
- link l_lfarm: geometry visual mesh filename=mesh/r_hand.obj
- link l_lglut: geometry visual mesh filename=mesh/l_lglut.obj
- link l_lleg: geometry visual mesh filename=mesh/l_lleg.obj
- link l_scap: geometry visual mesh filename=mesh/r_scap.obj
- link l_talus: geometry visual mesh filename=mesh/l_talus.obj
- link l_uarm: geometry visual mesh filename=mesh/r_uarm.obj
- link l_ufarm: geometry visual mesh filename=mesh/r_farm.obj
- link l_uglut: geometry visual mesh filename=mesh/l_uglut.obj
- link l_uleg: geometry visual mesh filename=mesh/l_uleg.obj
- link ltorso: geometry visual mesh filename=mesh/ltorso.obj
- link mtorso: geometry visual mesh filename=mesh/mtorso.obj
- link pelvis: geometry visual mesh filename=mesh/pelvis.obj
- link r_clav: geometry visual mesh filename=mesh/r_clav.obj
- link r_foot: geometry visual mesh filename=mesh/r_foot.obj
- link r_larm: geometry visual mesh filename=mesh/r_larm.obj
- link r_lfarm: geometry visual mesh filename=mesh/r_hand.obj
- link r_lglut: geometry visual mesh filename=mesh/r_lglut.obj
- link r_lleg: geometry visual mesh filename=mesh/r_lleg.obj
- link r_scap: geometry visual mesh filename=mesh/r_scap.obj
- link r_talus: geometry visual mesh filename=mesh/r_talus.obj
- link r_uarm: geometry visual mesh filename=mesh/r_uarm.obj
- link r_ufarm: geometry visual mesh filename=mesh/r_farm.obj
- link r_uglut: geometry visual mesh filename=mesh/r_uglut.obj
- link r_uleg: geometry visual mesh filename=mesh/r_uleg.obj
- link utorso: geometry visual mesh filename=mesh/utorso.obj

File: DojoEnvironments/src/panda/deps/panda_end_effector.urdf (robot description, URDF)
Before this commit: robot panda, 12 links, 11 joints
Links:
- link finger1: geometry collision mesh filename=mesh/collision/finger.stl; visual mesh filename=mesh/visual/finger.dae
- link finger2: geometry collision mesh filename=mesh/collision/finger.stl; visual mesh filename=mesh/visual/finger.dae
- link link0: geometry collision mesh filename=mesh/collision/link0.stl; visual mesh filename=mesh/visual/link0.dae
- link link1: geometry collision mesh filename=mesh/collision/link1.stl; visual mesh filename=mesh/visual/link1.dae
- link link2: geometry collision mesh filename=mesh/collision/link2.stl; visual mesh filename=mesh/visual/link2.dae
- link link3: geometry collision mesh filename=mesh/collision/link3.stl; visual mesh filename=mesh/visual/link3.dae
- link link4: geometry collision mesh filename=mesh/collision/link4.stl; visual mesh filename=mesh/visual/link4.dae
- link link5: geometry collision mesh filename=mesh/collision/link5.stl; visual mesh filename=mesh/visual/link5.dae
- link link6: geometry collision mesh filename=mesh/collision/link6.stl; visual mesh filename=mesh/visual/link6.dae
- link link7: geometry collision mesh filename=mesh/collision/link7.stl; visual mesh filename=mesh/visual/link7.dae
- link link8: geometry collision mesh filename=mesh/collision/hand.stl; visual mesh filename=mesh/visual/hand.dae

File: DojoEnvironments/src/panda/deps/panda_no_end_effector.urdf (robot description, URDF)
Before this commit: robot panda, 9 links, 8 joints
Links:
- link link0: geometry collision mesh filename=mesh/collision/link0.stl; visual mesh filename=mesh/visual/link0.dae
- link link1: geometry collision mesh filename=mesh/collision/link1.stl; visual mesh filename=mesh/visual/link1.dae
- link link2: geometry collision mesh filename=mesh/collision/link2.stl; visual mesh filename=mesh/visual/link2.dae
- link link3: geometry collision mesh filename=mesh/collision/link3.stl; visual mesh filename=mesh/visual/link3.dae
- link link4: geometry collision mesh filename=mesh/collision/link4.stl; visual mesh filename=mesh/visual/link4.dae
- link link5: geometry collision mesh filename=mesh/collision/link5.stl; visual mesh filename=mesh/visual/link5.dae
- link link6: geometry collision mesh filename=mesh/collision/link6.stl; visual mesh filename=mesh/visual/link6.dae
- link link7: geometry collision mesh filename=mesh/collision/link7.stl; visual mesh filename=mesh/visual/link7.dae

File: DojoEnvironments/src/quadruped/deps/quadruped.urdf (robot description, URDF)
Before this commit: robot a1_description, 13 links, 12 joints
Links:
- link FL_calf: geometry collision box size=0.2 0.016 0.016; visual mesh filename=mesh/calf.dae scale=1 1 1
- link FL_hip: geometry collision cylinder length=0.04 radius=0.046; visual mesh filename=mesh/hip.dae scale=1 1 1
- link FL_thigh: geometry collision box size=0.2 0.0245 0.034; visual mesh filename=mesh/thigh.dae scale=1 1 1
- link FR_calf: geometry collision box size=0.2 0.016 0.016; visual mesh filename=mesh/calf.dae scale=1 1 1
- link FR_hip: geometry collision cylinder length=0.04 radius=0.046; visual mesh filename=mesh/hip.dae scale=1 1 1
- link FR_thigh: geometry collision box size=0.2 0.0245 0.034; visual mesh filename=mesh/thigh_mirror.dae scale=1 1 1
- link RL_calf: geometry collision box size=0.2 0.016 0.016; visual mesh filename=mesh/calf.dae scale=1 1 1
- link RL_hip: geometry collision cylinder length=0.04 radius=0.046; visual mesh filename=mesh/hip.dae scale=1 1 1
- link RL_thigh: geometry collision box size=0.2 0.0245 0.034; visual mesh filename=mesh/thigh.dae scale=1 1 1
- link RR_calf: geometry collision box size=0.2 0.016 0.016; visual mesh filename=mesh/calf.dae scale=1 1 1
- link RR_hip: geometry collision cylinder length=0.04 radius=0.046; visual mesh filename=mesh/hip.dae scale=1 1 1
- link RR_thigh: geometry collision box size=0.2 0.0245 0.034; visual mesh filename=mesh/thigh_mirror.dae scale=1 1 1
- link trunk: geometry collision box size=0.267 0.194 0.114; visual mesh filename=mesh/trunk.dae scale=1 1 1

File: DojoEnvironments/src/quadruped/deps/quadruped_ones.urdf (robot description, URDF)
Before this commit: robot a1_description, 14 links, 13 joints
Links:
- link FL_calf: geometry collision box size=0.2 0.016 0.016; visual mesh filename=mesh/calf.dae scale=1 1 1
- link FL_hip: geometry collision cylinder length=0.04 radius=0.046; visual mesh filename=mesh/hip.dae scale=1 1 1
- link FL_thigh: geometry collision box size=0.2 0.0245 0.034; visual mesh filename=mesh/thigh.dae scale=1 1 1
- link FR_calf: geometry collision box size=0.2 0.016 0.016; visual mesh filename=mesh/calf.dae scale=1 1 1
- link FR_hip: geometry collision cylinder length=0.04 radius=0.046; visual mesh filename=mesh/hip.dae scale=1 1 1
- link FR_thigh: geometry collision box size=0.2 0.0245 0.034; visual mesh filename=mesh/thigh_mirror.dae scale=1 1 1
- link RL_calf: geometry collision box size=0.2 0.016 0.016; visual mesh filename=mesh/calf.dae scale=1 1 1
- link RL_hip: geometry collision cylinder length=0.04 radius=0.046; visual mesh filename=mesh/hip.dae scale=1 1 1
- link RL_thigh: geometry collision box size=0.2 0.0245 0.034; visual mesh filename=mesh/thigh.dae scale=1 1 1
- link RR_calf: geometry collision box size=0.2 0.016 0.016; visual mesh filename=mesh/calf.dae scale=1 1 1
- link RR_hip: geometry collision cylinder length=0.04 radius=0.046; visual mesh filename=mesh/hip.dae scale=1 1 1
- link RR_thigh: geometry collision box size=0.2 0.0245 0.034; visual mesh filename=mesh/thigh_mirror.dae scale=1 1 1
- link trunk: geometry collision box size=0.267 0.194 0.114; visual mesh filename=mesh/trunk.dae scale=1 1 1

File: DojoEnvironments/src/quadruped/deps/quadruped_simple.urdf (robot description, URDF)
Before this commit: robot a1_description, 14 links, 13 joints
Links:
- link FL_calf: geometry collision box size=0.2 0.016 0.016; visual mesh filename=mesh/calf.dae scale=1 1 1
- link FL_hip: geometry collision cylinder length=0.04 radius=0.046; visual mesh filename=mesh/hip.dae scale=1 1 1
- link FL_thigh: geometry collision box size=0.2 0.0245 0.034; visual mesh filename=mesh/thigh.dae scale=1 1 1
- link FR_calf: geometry collision box size=0.2 0.016 0.016; visual mesh filename=mesh/calf.dae scale=1 1 1
- link FR_hip: geometry collision cylinder length=0.04 radius=0.046; visual mesh filename=mesh/hip.dae scale=1 1 1
- link FR_thigh: geometry collision box size=0.2 0.0245 0.034; visual mesh filename=mesh/thigh_mirror.dae scale=1 1 1
- link RL_calf: geometry collision box size=0.2 0.016 0.016; visual mesh filename=mesh/calf.dae scale=1 1 1
- link RL_hip: geometry collision cylinder length=0.04 radius=0.046; visual mesh filename=mesh/hip.dae scale=1 1 1
- link RL_thigh: geometry collision box size=0.2 0.0245 0.034; visual mesh filename=mesh/thigh.dae scale=1 1 1
- link RR_calf: geometry collision box size=0.2 0.016 0.016; visual mesh filename=mesh/calf.dae scale=1 1 1
- link RR_hip: geometry collision cylinder length=0.04 radius=0.046; visual mesh filename=mesh/hip.dae scale=1 1 1
- link RR_thigh: geometry collision box size=0.2 0.0245 0.034; visual mesh filename=mesh/thigh_mirror.dae scale=1 1 1
- link trunk: geometry collision box size=0.267 0.194 0.114; visual mesh filename=mesh/trunk.dae scale=1 1 1

File: DojoEnvironments/src/rexhopper/deps/rexhopper.urdf (robot description, URDF)
Before this commit: robot rexhopper, 8 links, 7 joints
Links:
- link base_link: geometry collision mesh filename=mesh/base_link.obj; visual mesh filename=mesh/base_link.obj
- link link0: geometry collision mesh filename=mesh/link0.obj; visual mesh filename=mesh/link0.obj
- link link1: geometry collision mesh filename=mesh/link1.obj; visual mesh filename=mesh/link1.obj
- link link2: geometry collision mesh filename=mesh/link2.obj; visual mesh filename=mesh/link2.obj
- link link3: geometry collision mesh filename=mesh/link3.obj; visual mesh filename=mesh/link3.obj
- link rw0: geometry collision mesh filename=mesh/rw0.obj; visual mesh filename=mesh/rw0.obj
- link rw1: geometry collision mesh filename=mesh/rw1.obj; visual mesh filename=mesh/rw1.obj
- link rwz: geometry collision mesh filename=mesh/rwz.obj; visual mesh filename=mesh/rwz.obj

File: DojoEnvironments/src/rexhopper/deps/rexhopper0.urdf (robot description, URDF)
Before this commit: robot rexhopper, 8 links, 7 joints
Links:
- link base_link: geometry collision mesh filename=mesh/base_link.obj; visual mesh filename=mesh/base_link.obj
- link link0: geometry collision mesh filename=mesh/link0.obj; visual mesh filename=mesh/link0.obj
- link link1: geometry collision mesh filename=mesh/link1.obj; visual mesh filename=mesh/link1.obj
- link link2: geometry collision mesh filename=mesh/link2.obj; visual mesh filename=mesh/link2.obj
- link link3: geometry collision mesh filename=mesh/link3.obj; visual mesh filename=mesh/link3.obj
- link rw0: geometry collision mesh filename=mesh/rw0.obj; visual mesh filename=mesh/rw0.obj
- link rw1: geometry collision mesh filename=mesh/rw1.obj; visual mesh filename=mesh/rw1.obj
- link rwz: geometry collision mesh filename=mesh/rwz.obj; visual mesh filename=mesh/rwz.obj

File: DojoEnvironments/src/rexhopper/deps/rexhopper1.urdf (robot description, URDF)
Before this commit: robot rexhopper, 2 links, 1 joints
Links:
- link base_link: geometry collision mesh filename=mesh/base_link.obj; visual mesh filename=mesh/base_link.obj
- link rw1: geometry collision mesh filename=mesh/rw1.obj; visual mesh filename=mesh/rw1.obj

File: DojoEnvironments/src/rexhopper/deps/rexhopper2.urdf (robot description, URDF)
Before this commit: robot rexhopper, 5 links, 4 joints
Links:
- link base_link: geometry collision mesh filename=mesh/base_link.obj; visual mesh filename=mesh/base_link.obj
- link link0: geometry collision mesh filename=mesh/link0.obj; visual mesh filename=mesh/link0.obj
- link link1: geometry collision mesh filename=mesh/link1.obj; visual mesh filename=mesh/link1.obj
- link link2: geometry collision mesh filename=mesh/link2.obj; visual mesh filename=mesh/link2.obj
- link link3: geometry collision mesh filename=mesh/link3.obj; visual mesh filename=mesh/link3.obj

File: DojoEnvironments/src/rexhopper/deps/rexhopper3.urdf (robot description, URDF)
Before this commit: robot rexhopper, 2 links, 1 joints
Links:
- link link2: geometry collision mesh filename=mesh/link2.obj; visual mesh filename=mesh/link2.obj
- link link3: geometry collision mesh filename=mesh/link3.obj; visual mesh filename=mesh/link3.obj
