Commit message: get DojoEnvironment tests to pass

File: DojoEnvironments/src/rexhopper/deps/rexhopper_base.urdf (robot description, URDF)
Before this commit: robot rexhopper, 8 links, 7 joints
Links:
- link base_link: geometry collision mesh filename=mesh/base_link.obj; visual mesh filename=mesh/base_link.obj
- link link0: geometry collision mesh filename=mesh/link0.obj; visual mesh filename=mesh/link0.obj
- link link1: geometry collision mesh filename=mesh/link1.obj; visual mesh filename=mesh/link1.obj
- link link2: geometry collision mesh filename=mesh/link2.obj; visual mesh filename=mesh/link2.obj
- link link3: geometry collision mesh filename=mesh/link3.obj; visual mesh filename=mesh/link3.obj
- link rw0: geometry collision mesh filename=mesh/rw0.obj; visual mesh filename=mesh/rw0.obj
- link rw1: geometry collision mesh filename=mesh/rw1.obj; visual mesh filename=mesh/rw1.obj
- link rwz: geometry collision mesh filename=mesh/rwz.obj; visual mesh filename=mesh/rwz.obj

File: DojoEnvironments/src/rexhopper/deps/rexhopper_damper.urdf (robot description, URDF)
Before this commit: robot rexhopper, 2 links, 1 joints
Links:
- link base_link: geometry collision mesh filename=mesh/base_link.obj; visual mesh filename=mesh/base_link.obj
- link rw0: geometry collision mesh filename=mesh/rw0.obj; visual mesh filename=mesh/rw0.obj

File: DojoEnvironments/src/rexhopper/deps/rexhopper_fixed.urdf (robot description, URDF)
Before this commit: robot rexhopper, 8 links, 7 joints
Links:
- link base_link: geometry collision mesh filename=mesh/base_link.obj; visual mesh filename=mesh/base_link.obj
- link link0: geometry collision mesh filename=mesh/link0.obj; visual mesh filename=mesh/link0.obj
- link link1: geometry collision mesh filename=mesh/link1.obj; visual mesh filename=mesh/link1.obj
- link link2: geometry collision mesh filename=mesh/link2.obj; visual mesh filename=mesh/link2.obj
- link link3: geometry collision mesh filename=mesh/link3.obj; visual mesh filename=mesh/link3.obj
- link rw0: geometry collision mesh filename=mesh/rw0.obj; visual mesh filename=mesh/rw0.obj
- link rw1: geometry collision mesh filename=mesh/rw1.obj; visual mesh filename=mesh/rw1.obj
- link rwz: geometry collision mesh filename=mesh/rwz.obj; visual mesh filename=mesh/rwz.obj
