Commit message: Update youbot arm URDF

File: DojoEnvironments/src/youbot/deps/youbot_arm_only_fixed_gripper.urdf (robot description, URDF)
Before this commit: robot youbot, 9 links, 8 joints
Joints:
- joint gripper_finger_joint_l: type prismatic -> fixed
- joint gripper_finger_joint_r: type prismatic -> fixed
