Commit message: Update youbot URDFs

File: DojoEnvironments/src/youbot/deps/youbot.urdf (robot description, URDF)
Before this commit: robot youbot, 21 links, 20 joints
Links:
- removed link caster_link_bl
- removed link caster_link_br
- removed link caster_link_fl
- removed link caster_link_fr
- link wheel_link_bl: mass 1.4 -> 1.5
- link wheel_link_br: mass 1.4 -> 1.5
- link wheel_link_fl: mass 1.4 -> 1.5
- link wheel_link_fr: mass 1.4 -> 1.5
Joints:
- removed joint caster_joint_bl
- removed joint caster_joint_br
- removed joint caster_joint_fl
- removed joint caster_joint_fr
- joint base_footprint_joint: axis (none) -> 0 0 1; origin xyz=0 0 0 rpy=0 0 0 -> xyz=0 0 0.083 rpy=0 0 0; type fixed -> planaraxis
- joint wheel_joint_bl: origin xyz=0.0 0.0 0.0 rpy=0 0 0 -> xyz=-0.228 0.158 -0.034 rpy=0 0 0; parent caster_link_bl -> base_link
- joint wheel_joint_br: origin xyz=0.0 0.0 0.0 rpy=0 0 0 -> xyz=-0.228 -0.158 -0.034 rpy=0 0 0; parent caster_link_br -> base_link
- joint wheel_joint_fl: origin xyz=0.0 0.0 0.0 rpy=0 0 0 -> xyz=0.228 0.158 -0.034 rpy=0 0 0; parent caster_link_fl -> base_link
- joint wheel_joint_fr: origin xyz=0.0 0.0 0.0 rpy=0 0 0 -> xyz=0.228 -0.158 -0.034 rpy=0 0 0; parent caster_link_fr -> base_link

File: DojoEnvironments/src/youbot/deps/youbot_base_only.urdf (robot description, URDF)
Before this commit: robot youbot, 11 links, 10 joints
Links:
- removed link caster_link_bl
- removed link caster_link_br
- removed link caster_link_fl
- removed link caster_link_fr
- link wheel_link_bl: mass 1.4 -> 1.5
- link wheel_link_br: mass 1.4 -> 1.5
- link wheel_link_fl: mass 1.4 -> 1.5
- link wheel_link_fr: mass 1.4 -> 1.5
Joints:
- removed joint caster_joint_bl
- removed joint caster_joint_br
- removed joint caster_joint_fl
- removed joint caster_joint_fr
- joint base_footprint_joint: axis (none) -> 0 0 1; origin xyz=0 0 0 rpy=0 0 0 -> xyz=0 0 0.083 rpy=0 0 0; type fixed -> planaraxis
- joint wheel_joint_bl: origin xyz=0.0 0.0 0.0 rpy=0 0 0 -> xyz=-0.228 0.158 -0.034 rpy=0 0 0; parent caster_link_bl -> base_link
- joint wheel_joint_br: origin xyz=0.0 0.0 0.0 rpy=0 0 0 -> xyz=-0.228 -0.158 -0.034 rpy=0 0 0; parent caster_link_br -> base_link
- joint wheel_joint_fl: origin xyz=0.0 0.0 0.0 rpy=0 0 0 -> xyz=0.228 0.158 -0.034 rpy=0 0 0; parent caster_link_fl -> base_link
- joint wheel_joint_fr: origin xyz=0.0 0.0 0.0 rpy=0 0 0 -> xyz=0.228 -0.158 -0.034 rpy=0 0 0; parent caster_link_fr -> base_link
