Commit message: wip

File: DojoEnvironments/src/panda/deps/panda_end_effector.urdf (robot description, URDF)
Before this commit: robot panda, 12 links, 11 joints
Links:
- removed link world
Joints:
- removed joint joint0

File: DojoEnvironments/src/panda/deps/panda_no_end_effector.urdf (robot description, URDF)
Before this commit: robot panda, 8 links, 7 joints
Links:
- removed link world
Joints:
- removed joint joint0

File: DojoEnvironments/src/panda/deps/panda_original.urdf (robot description, URDF)
Before this commit: robot panda, 11 links, 10 joints
Links:
- removed link world
Joints:
- removed joint panda_joint_panda_mount
