Commit message: Initial Environments restructuring

File: DojoEnvironments/src/hopper/deps/hopper.urdf (robot description, URDF)
Before this commit: robot hopper, 3 links, 2 joints
Links:
- added link foot, mass 5.08938; collision capsule length=0.39 radius=0.06; visual capsule length=0.39 radius=0.06
- added link leg, mass 2.71433; collision capsule length=0.5 radius=0.04; visual capsule length=0.5 radius=0.04
Joints:
- added joint foot: type revolute, parent leg, child foot, origin xyz=0.00000 0.00000 -0.50000 rpy=0.00000 0.00000 0.00000, axis 0.00000 1.00000 0.00000
- added joint leg: type revolute, parent thigh, child leg, origin xyz=0.0000 0.00000 -0.45000 rpy=0.00000 0.00000 0.00000, axis 0.00000 1.00000 0.00000
