Commit message: Small changes and fixes

File: DojoEnvironments/src/mechanisms/uuv/dependencies/mini_tortuga.urdf (robot description, URDF)
Before this commit: robot mini_tortuga, 7 links, 6 joints
Links:
- added link origin, mass 1
Joints:
- added joint floating_base: type floating, parent origin, child base_link, origin xyz=0 0 0 rpy=0 0 0

File: DojoEnvironments/src/mechanisms/uuv/dependencies/mini_tortuga_fixed_rotors.urdf (robot description, URDF)
Before this commit: robot mini_tortuga, 7 links, 6 joints
Links:
- added link origin, mass 1
Joints:
- added joint floating_base: type floating, parent origin, child base_link, origin xyz=0 0 0 rpy=0 0 0

File: DojoEnvironments/src/mechanisms/youbot/dependencies/youbot.urdf (robot description, URDF)
Before this commit: robot youbot, 17 links, 16 joints
Joints:
- joint arm_joint_1: origin xyz=0.024 0 0.096 rpy=0 0 2.9670597283903604 -> xyz=0.024 0 0.096 rpy=0 0 0
- joint arm_joint_2: origin xyz=0.033 0 0.019 rpy=0 -1.1344640137963142 0 -> xyz=0.033 0 0.019 rpy=0 0 0
- joint arm_joint_3: origin xyz=0.000 0.000 0.155 rpy=0 2.548180707911721 0 -> xyz=0.000 0.000 0.155 rpy=0 0 0
- joint arm_joint_4: origin xyz=0.000 0.000 0.135 rpy=0 -1.7889624832941877 0 -> xyz=0.000 0.000 0.135 rpy=0 0 0
- joint arm_joint_5: origin xyz=-0.002 0 0.130 rpy=0 0 2.9234264970905017 -> xyz=-0.002 0 0.130 rpy=0 0 0
